Commit message: Update v1.1

File: agv_description/urdf/agv.urdf.xacro (robot description, xacro)
@@ -1,4 +1,4 @@
 <?xml version="1.0"?>
-<robot name="AGV" xmlns:xacro="http://ros.org/wiki/xacro">
+<robot name="AGV-OTA" xmlns:xacro="http://ros.org/wiki/xacro">
 	<xacro:include filename="$(find agv_description)/urdf/agv_base.urdf.xacro"/>
 	<xacro:include filename="$(find agv_description)/urdf/inertia_tensors.urdf.xacro"/>

File: agv_description/urdf/agv_base.urdf.xacro (robot description, xacro)
@@ -7,11 +7,12 @@
         <origin xyz="0 0 -0.1625" rpy=" 0 0 0"/>
         <geometry>
-        <mesh filename="package://agv_description/meshes/OTAv07_meshes/OTA-v0.7.stl" scale="0.001 0.001 0.001"/>
+          <mesh filename="package://agv_description/meshes/OTAv07_meshes/OTA-v0.7.stl" scale="0.001 0.001 0.001"/>
         </geometry>
       </visual>
       <collision>
-        <origin xyz="0 0 -0.1625" rpy=" 0 0 0"/>
+        <origin xyz="0 0 0.011" rpy=" 0 0 0"/>
         <geometry>
-          <mesh filename="package://agv_description/meshes/OTAv07_meshes/OTA-v0.7.stl" scale="0.001 0.001 0.001"/>
+          <!--<mesh filename="package://agv_description/meshes/OTAv07_meshes/OTA-v0.7.stl" scale="0.001 0.001 0.001"/> -->
+          <box size="1.02 0.72 0.29"/>
         </geometry>
       </collision>
@@ -29,10 +30,10 @@
         </geometry>
       </visual>
-      <collision>
+      <!--<collision>
         <origin xyz="0 0 0.0" rpy="1.570796 0 -1.570796"/>
         <geometry>
           <mesh filename="package://agv_description/meshes/OTAv07_meshes/S30B-XXXXXX.stl" scale="0.001 0.001 0.001"/>
         </geometry>
-      </collision>
+      </collision>  -->
     </link>
     <joint name="scan_joint" type="fixed">
@@ -45,4 +46,5 @@
       <material value="Gazebo/DarkGray"/>
       <sensor type="ray" name="laser_scan">
+      	<tf_prefix></tf_prefix>
         <pose>0 0 0 0 0 0</pose>
         <visualize>false</visualize>
@@ -128,6 +130,6 @@
           <updateRate>0.0</updateRate>
           <cameraName>camera</cameraName>
-          <imageTopicName>/camera/image_raw</imageTopicName>
-          <cameraInfoTopicName>/camera/camera_info</cameraInfoTopicName>
+          <imageTopicName>image_raw</imageTopicName>
+          <cameraInfoTopicName>camera_info</cameraInfoTopicName>
           <frameName>zed_camera</frameName>
           <hackBaseline>0.07</hackBaseline>

File: agv_description/urdf/agv_plugin.urdf.xacro (robot description, xacro)
@@ -5,5 +5,4 @@
   	<gazebo>
          <plugin name="joint_state_publisher" filename="libgazebo_ros_joint_state_publisher.so">
-            <robotNamespace></robotNamespace>
             <jointName>caster_front_left_joint,caster_front_right_joint,caster_back_left_joint,caster_back_right_joint,caster_front_left_wheel_joint,caster_front_right_wheel_joint,caster_back_left_wheel_joint,caster_back_right_wheel_joint</jointName>
             <updateRate>10.0</updateRate>
@@ -17,5 +16,4 @@
       <plugin name="differential_drive_controller" filename="libgazebo_ros_diff_drive.so">
         <rosDebugLevel>Debug</rosDebugLevel>
-        <robotNamespace>/</robotNamespace>
         <publishWheelTF>false</publishWheelTF>
         <publishOdomTF>true</publishOdomTF>
